File: hardware/base-pcb/gifu-creation-koubou.kicad_sch (KiCad schematic)
At the start: 110 parts, among them J1 Jack-DC, J10 Conn_01x01, J11 Conn_01x01, J2 Conn_01x03, J3 Conn_01x03, J4 Conn_01x01, J5 Conn_01x01, J6 Conn_01x03, J7 AudioJack3, J8 Conn_01x01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

Commit message: reorganize folder structure, add module circuits
Other:
- company: (none) -> Kinoshita Laboratory
- title: (none) -> Gifu Creation Koubou Teaching Material
Changed lines of the file:
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@@
 (kicad_sch (version 20211123) (generator eeschema)
   (paper "A2")
+  (title_block
+    (title "Gifu Creation Koubou Teaching Material")
+    (date "2022-08-21")
+    (rev "20220820")
+    (company "Kinoshita Laboratory")
+  )
   (junction (at 73.66 248.92) (diameter 0) (color 0 0 0 0)
   )
